File: ai03-pcb-guide.kicad_pcb (KiCad board)
At the start: 2 copper layers, 92.1 x 38.1 mm, 24 parts, among them SW1 SW_Push, U1 ATmega32U4-AU, Y1 16MHz

Commit message: Prettify pcb
Parts:
- moved D1 4.19 mm to (140.7, 34.3)
- moved MX1 4.19 mm to (132.3, 34.9)
- moved D2 4.19 mm to (140.6, 53.0)
- moved D3 4.19 mm to (159.6, 34.0)
- moved D4 4.19 mm to (159.9, 53.3)
- moved MX3 4.19 mm to (151.4, 34.8)
- moved MX4 4.19 mm to (151.5, 54.0)
- moved MX2 4.19 mm to (132.5, 54.0)
Routing:
- net COL0: track 38.2 -> 33.9 mm
- net COL1: track 63.4 -> 59.2 mm
- net ROW0: track 54.2 -> 50.1 mm
- net ROW1: track 54.6 -> 52.6 mm
- added copper zone on B.Cu, net GND
Other:
- board size 92.1 x 38.1 mm -> 87.9 x 38.2 mm
- board text added: "Hello World"
